Commit message: xacro files chagened

File: src/gp12_gazebo/urdf/gp12.xacro (robot description, xacro)
@@ -1,91 +1,5 @@
 <?xml version="1.0" ?>
 <robot name="motoman_gp12" xmlns:xacro="http://ros.org/wiki/xacro">
-    <!-- <xacro:include filename="$(find motoman_gp12_support)/urdf/gp12_macro.xacro" />
-    <xacro:motoman_gp12 prefix=""/> -->
-    <!-- Transmissions for ros2_control simulation -->
-<transmission name="trans_s">
-  <type>transmission_interface/SimpleTransmission</type>
-  <joint name="joint_s">
-    <hardwareInterface>hardware_interface/PositionOnlyJointInterface</hardwareInterface>
-  </joint>
-  <actuator name="motor_s">
-    <mechanicalReduction>1</mechanicalReduction>
-  </actuator>
-</transmission>
-<transmission name="trans_l">
-  <type>transmission_interface/SimpleTransmission</type>
-  <joint name="joint_l">
-    <hardwareInterface>hardware_interface/PositionOnlyJointInterface</hardwareInterface>
-  </joint>
-  <actuator name="motor_l">
-    <mechanicalReduction>1</mechanicalReduction>
-  </actuator>
-</transmission>
-<!-- Repeat for joint_u, joint_r, joint_b, joint_t -->
-<!-- Example for joint_u -->
-<transmission name="trans_u">
-  <type>transmission_interface/SimpleTransmission</type>
-  <joint name="joint_u">
-    <hardwareInterface>hardware_interface/PositionOnlyJointInterface</hardwareInterface>
-  </joint>
-  <actuator name="motor_u">
-    <mechanicalReduction>1</mechanicalReduction>
-  </actuator>
-</transmission>
-<!-- ... add joint_r, joint_b, joint_t similarly -->
-<!-- ros2_control transmissions for Gazebo simulation -->
-<transmission name="trans_joint_s">
-  <type>transmission_interface/SimpleTransmission</type>
-  <joint name="joint_s">
-    <hardwareInterface>hardware_interface/PositionOnlyJointInterface</hardwareInterface>
-  </joint>
-  <actuator name="motor_s">
-    <mechanicalReduction>1</mechanicalReduction>
-  </actuator>
-</transmission>
-<transmission name="trans_joint_l">
-  <type>transmission_interface/SimpleTransmission</type>
-  <joint name="joint_l">
-    <hardwareInterface>hardware_interface/PositionOnlyJointInterface</hardwareInterface>
-  </joint>
-  <actuator name="motor_l">
-    <mechanicalReduction>1</mechanicalReduction>
-  </actuator>
-</transmission>
-<transmission name="trans_joint_u">
-  <type>transmission_interface/SimpleTransmission</type>
-  <joint name="joint_u">
-    <hardwareInterface>hardware_interface/PositionOnlyJointInterface</hardwareInterface>
-  </joint>
-  <actuator name="motor_u">
-    <mechanicalReduction>1</mechanicalReduction>
-  </actuator>
-</transmission>
-<transmission name="trans_joint_r">
-  <type>transmission_interface/SimpleTransmission</type>
-  <joint name="joint_r">
-    <hardwareInterface>hardware_interface/PositionOnlyJointInterface</hardwareInterface>
-  </joint>
-  <actuator name="motor_r">
-    <mechanicalReduction>1</mechanicalReduction>
-  </actuator>
-</transmission>
-<transmission name="trans_joint_b">
-  <type>transmission_interface/SimpleTransmission</type>
-  <joint name="joint_b">
-    <hardwareInterface>hardware_interface/PositionOnlyJointInterface</hardwareInterface>
-  </joint>
-  <actuator name="motor_b">
-    <mechanicalReduction>1</mechanicalReduction>
-  </actuator>
-</transmission>
-<transmission name="trans_joint_t">
-  <type>transmission_interface/SimpleTransmission</type>
-  <joint name="joint_t">
-    <hardwareInterface>hardware_interface/PositionOnlyJointInterface</hardwareInterface>
-  </joint>
-  <actuator name="motor_t">
-    <mechanicalReduction>1</mechanicalReduction>
-  </actuator>
-</transmission>
+    <xacro:include filename="$(find motoman_gp12_support)/urdf/gp12_macro.xacro" />
+    <xacro:motoman_gp12 prefix=""/>
 </robot>

Commit message: fixed erros

File: src/gp12_gazebo/urdf/gp12.xacro (robot description, xacro)
@@ -1,5 +1,5 @@
 <?xml version="1.0" ?>
 <robot name="motoman_gp12" xmlns:xacro="http://ros.org/wiki/xacro">
-    <xacro:include filename="$(find motoman_gp12_support)/urdf/gp12_macro.xacro" />
+    <xacro:include filename="$(find gp12_gazebo)/urdf/gp12_macro.xacro" />
     <xacro:motoman_gp12 prefix=""/>
 </robot>

File: src/gp12_gazebo/urdf/gp12_macro.xacro (robot description, xacro)
@@ -2,10 +2,10 @@
 <robot xmlns:xacro="http://ros.org/wiki/xacro">
 <xacro:macro name="motoman_gp12" params="prefix">
-    <xacro:include filename="$(find motoman_resources)/urdf/common_materials.xacro"/>
+    <xacro:include filename="$(find gp12_gazebo)/urdf/common_materials.xacro"/>
     <!-- link list -->
     <link name="${prefix}base_link">
         <visual>
             <geometry>
-                <mesh filename="package://motoman_gp12_support/meshes/visual/gp12_base_link.stl"/>
+                <mesh filename="package://gp12_gazebo/meshes/visual/gp12_base_link.stl"/>
             </geometry>
             <xacro:material_yaskawa_blue/>
@@ -13,5 +13,5 @@
         <collision>
             <geometry>
-                <mesh filename="package://motoman_gp12_support/meshes/collision/gp12_base_link.stl"/>
+                <mesh filename="package://gp12_gazebo/meshes/collision/gp12_base_link.stl"/>
             </geometry>
         </collision>
@@ -20,5 +20,5 @@
         <visual>
             <geometry>
-                <mesh filename="package://motoman_gp12_support/meshes/visual/gp12_link_1_s.stl"/>
+                <mesh filename="package://gp12_gazebo/meshes/visual/gp12_link_1_s.stl"/>
             </geometry>
             <xacro:material_yaskawa_blue/>
@@ -26,5 +26,5 @@
         <collision>
             <geometry>
-                <mesh filename="package://motoman_gp12_support/meshes/collision/gp12_link_1_s.stl"/>
+                <mesh filename="package://gp12_gazebo/meshes/collision/gp12_link_1_s.stl"/>
             </geometry>
         </collision>
@@ -33,5 +33,5 @@
         <visual>
             <geometry>
-                <mesh filename="package://motoman_gp12_support/meshes/visual/gp12_link_2_l.stl"/>
+                <mesh filename="package://gp12_gazebo/meshes/visual/gp12_link_2_l.stl"/>
             </geometry>
             <xacro:material_yaskawa_blue/>
@@ -39,5 +39,5 @@
         <collision>
             <geometry>
-                <mesh filename="package://motoman_gp12_support/meshes/collision/gp12_link_2_l.stl"/>
+                <mesh filename="package://gp12_gazebo/meshes/collision/gp12_link_2_l.stl"/>
             </geometry>
         </collision>
@@ -46,5 +46,5 @@
         <visual>
             <geometry>
-                <mesh filename="package://motoman_gp12_support/meshes/visual/gp12_link_3_u.stl"/>
+                <mesh filename="package://gp12_gazebo/meshes/visual/gp12_link_3_u.stl"/>
             </geometry>
             <xacro:material_yaskawa_blue/>
@@ -52,5 +52,5 @@
         <collision>
             <geometry>
-                <mesh filename="package://motoman_gp12_support/meshes/collision/gp12_link_3_u.stl"/>
+                <mesh filename="package://gp12_gazebo/meshes/collision/gp12_link_3_u.stl"/>
             </geometry>
         </collision>
@@ -59,5 +59,5 @@
         <visual>
             <geometry>
-                <mesh filename="package://motoman_gp12_support/meshes/visual/gp12_link_4_r.stl"/>
+                <mesh filename="package://gp12_gazebo/meshes/visual/gp12_link_4_r.stl"/>
             </geometry>
             <xacro:material_yaskawa_blue/>
@@ -65,5 +65,5 @@
         <collision>
             <geometry>
-                <mesh filename="package://motoman_gp12_support/meshes/collision/gp12_link_4_r.stl"/>
+                <mesh filename="package://gp12_gazebo/meshes/collision/gp12_link_4_r.stl"/>
             </geometry>
         </collision>
@@ -72,5 +72,5 @@
         <visual>
             <geometry>
-                <mesh filename="package://motoman_gp12_support/meshes/visual/gp12_link_5_b.stl"/>
+                <mesh filename="package://gp12_gazebo/meshes/visual/gp12_link_5_b.stl"/>
             </geometry>
             <xacro:material_yaskawa_blue/>
@@ -78,5 +78,5 @@
         <collision>
             <geometry>
-                <mesh filename="package://motoman_gp12_support/meshes/collision/gp12_link_5_b.stl"/>
+                <mesh filename="package://gp12_gazebo/meshes/collision/gp12_link_5_b.stl"/>
             </geometry>
         </collision>
@@ -85,5 +85,5 @@
         <visual>
             <geometry>
-                <mesh filename="package://motoman_gp12_support/meshes/visual/gp12_link_6_t.stl"/>
+                <mesh filename="package://gp12_gazebo/meshes/visual/gp12_link_6_t.stl"/>
             </geometry>
             <xacro:material_yaskawa_blue/>
@@ -91,5 +91,5 @@
         <collision>
             <geometry>
-                <mesh filename="package://motoman_gp12_support/meshes/collision/gp12_link_6_t.stl"/>
+                <mesh filename="package://gp12_gazebo/meshes/collision/gp12_link_6_t.stl"/>
             </geometry>
         </collision>
