Commit message: fixed the xacro file and switched to classic gazebo version

File: src/gp12_gazebo/urdf/gp12_macro.xacro (robot description, xacro)
@@ -5,4 +5,9 @@
     <!-- link list -->
     <link name="${prefix}base_link">
+        <inertial>
+            <mass value="15.0"/>  <!-- guess – adjust based on real robot if possible -->
+            <origin xyz="0 0 0.15" rpy="0 0 0"/>  <!-- rough CoM along link -->
+            <inertia ixx="0.5" ixy="0" ixz="0" iyy="0.5" iyz="0" izz="0.1"/>
+        </inertial>
         <visual>
             <geometry>
@@ -139,26 +144,72 @@
         <limit lower="-7.9412" upper="7.9412" effort="33.30" velocity="12.2143"/>
     </joint>
+     <ros2_control name="GP12System" type="system">
+      <hardware>
+        <plugin>gazebo_ros2_control/GazeboSystem</plugin>
+      </hardware>
+        <joint name="${prefix}joint_1_s">
+            <command_interface name="effort"/>
+            <state_interface name="position"/>
+            <state_interface name="velocity"/>
+            <state_interface name="effort"/>
+        </joint>
+        <joint name="${prefix}joint_2_l">
+            <command_interface name="effort"/>
+            <state_interface name="position"/>
+            <state_interface name="velocity"/>
+            <state_interface name="effort"/>
+        </joint>
+        <joint name="${prefix}joint_3_u">
+            <command_interface name="effort"/>
+            <state_interface name="position"/>
+            <state_interface name="velocity"/>
+            <state_interface name="effort"/>
+        </joint>
+        <joint name="${prefix}joint_4_r">
+            <command_interface name="effort"/>
+            <state_interface name="position"/>
+            <state_interface name="velocity"/>
+            <state_interface name="effort"/>
+        </joint>
+        <joint name="${prefix}joint_5_b">
+            <command_interface name="effort"/>
+            <state_interface name="position"/>
+            <state_interface name="velocity"/>
+            <state_interface name="effort"/>
+        </joint>
+        <joint name="${prefix}joint_6_t">
+            <command_interface name="effort"/>
+            <state_interface name="position"/>
+            <state_interface name="velocity"/>
+            <state_interface name="effort"/>
+        </joint>
+    </ros2_control>
     <!-- end of joint list -->
     <!-- ROS base_link to Robot Manufacturer World Coordinates transform -->
-    <link name="${prefix}base" />
+    <!-- <link name="${prefix}base" />
     <joint name="${prefix}base_link-base" type="fixed">
         <origin xyz="0 0 0.450" rpy="0 0 0"/>
         <parent link="${prefix}base_link"/>
         <child link="${prefix}base"/>
-    </joint>
+    </joint> -->
     <!-- ROS-Industrial 'flange' frame: attachment point for EEF models -->
-    <link name="${prefix}flange"/>
+    <!-- <link name="${prefix}flange"/>
     <joint name="${prefix}joint_6_t-flange" type="fixed">
       <origin xyz="0.100 0 0" rpy="0 0 0"/>
       <parent link="${prefix}link_6_t"/>
       <child link="${prefix}flange"/>
-    </joint>
+    </joint> -->
     <!-- ROS-Industrial 'tool0' frame: all-zeros tool frame -->
-    <link name="${prefix}tool0"/>
+    <!-- <link name="${prefix}tool0"/>
     <joint name="${prefix}flange-tool0" type="fixed">
       <origin xyz="0 0 0" rpy="3.1415926 -1.570796 0"/>
       <parent link="${prefix}flange"/>
       <child link="${prefix}tool0"/>
-    </joint>
+    </joint> -->
+    <gazebo>
+      <plugin name="gazebo_ros2_control" filename="libgazebo_ros2_control.so">
+        <parameters>$(find gp12_gazebo)/config/gp12_controllers.yaml</parameters>
+      </plugin>
+    </gazebo>
     </xacro:macro>
 </robot>

Commit message: add rviz

File: src/gp12_gazebo/urdf/gp12_macro.xacro (robot description, xacro)
@@ -187,24 +187,24 @@
     <!-- end of joint list -->
     <!-- ROS base_link to Robot Manufacturer World Coordinates transform -->
-    <!-- <link name="${prefix}base" />
+    <link name="${prefix}base" />
     <joint name="${prefix}base_link-base" type="fixed">
         <origin xyz="0 0 0.450" rpy="0 0 0"/>
         <parent link="${prefix}base_link"/>
         <child link="${prefix}base"/>
-    </joint> -->
+    </joint>
     <!-- ROS-Industrial 'flange' frame: attachment point for EEF models -->
-    <!-- <link name="${prefix}flange"/>
+    <link name="${prefix}flange"/>
     <joint name="${prefix}joint_6_t-flange" type="fixed">
       <origin xyz="0.100 0 0" rpy="0 0 0"/>
       <parent link="${prefix}link_6_t"/>
       <child link="${prefix}flange"/>
-    </joint> -->
+    </joint>
     <!-- ROS-Industrial 'tool0' frame: all-zeros tool frame -->
-    <!-- <link name="${prefix}tool0"/>
+    <link name="${prefix}tool0"/>
     <joint name="${prefix}flange-tool0" type="fixed">
       <origin xyz="0 0 0" rpy="3.1415926 -1.570796 0"/>
       <parent link="${prefix}flange"/>
       <child link="${prefix}tool0"/>
-    </joint> -->
+    </joint>
     </xacro:macro>
 </robot>

Commit message: changes in xacro file

File: src/gp12_gazebo/urdf/gp12_macro.xacro (robot description, xacro)
@@ -23,4 +23,9 @@
     </link>
     <link name="${prefix}link_1_s">
+        <inertial>
+            <mass value="20.0"/>  <!-- guess -->
+            <origin xyz="0.08 0 0" rpy="0 0 0"/>  <!-- rough CoM -->
+            <inertia ixx="0.5" ixy="0" ixz="0" iyy="0.5" iyz="0" izz="0.1"/>
+        </inertial>
         <visual>
             <geometry>
@@ -36,4 +41,9 @@
     </link>
     <link name="${prefix}link_2_l">
+        <inertial>
+            <mass value="40.0"/>  <!-- guess -->
+            <origin xyz="0 0 0.307" rpy="0 0 0"/>  <!-- rough CoM -->
+            <inertia ixx="1.0" ixy="0" ixz="0" iyy="1.0" iyz="0" izz="0.2"/>
+        </inertial>
         <visual>
             <geometry>
@@ -49,4 +59,9 @@
     </link>
     <link name="${prefix}link_3_u">
+        <inertial>
+            <mass value="35.0"/>  <!-- guess -->
+            <origin xyz="0.32 0 0.1" rpy="0 0 0"/>  <!-- rough CoM -->
+            <inertia ixx="1.0" ixy="0" ixz="0" iyy="1.0" iyz="0" izz="0.2"/>
+        </inertial>
         <visual>
             <geometry>
@@ -62,4 +77,9 @@
     </link>
     <link name="${prefix}link_4_r">
+        <inertial>
+            <mass value="20.0"/>  <!-- guess -->
+            <origin xyz="0 0 0" rpy="0 0 0"/>  <!-- rough CoM -->
+            <inertia ixx="0.5" ixy="0" ixz="0" iyy="0.5" iyz="0" izz="0.1"/>
+        </inertial>
         <visual>
             <geometry>
@@ -75,4 +95,9 @@
     </link>
     <link name="${prefix}link_5_b">
+        <inertial>
+            <mass value="15.0"/>  <!-- guess -->
+            <origin xyz="0 0 0" rpy="0 0 0"/>  <!-- rough CoM -->
+            <inertia ixx="0.4" ixy="0" ixz="0" iyy="0.4" iyz="0" izz="0.1"/>
+        </inertial>
         <visual>
             <geometry>
@@ -88,4 +113,9 @@
     </link>
     <link name="${prefix}link_6_t">
+        <inertial>
+            <mass value="5.0"/>  <!-- guess -->
+            <origin xyz="0.05 0 0" rpy="0 0 0"/>  <!-- rough CoM -->
+            <inertia ixx="0.1" ixy="0" ixz="0" iyy="0.1" iyz="0" izz="0.05"/>
+        </inertial>
         <visual>
             <geometry>
