Commit message: removed gazebo

File: src/gp12_simulation/urdf/common_materials.xacro (robot description, xacro)
@@ -1,5 +1,5 @@
 <?xml version="1.0" ?>
 <robot xmlns:xacro="http://ros.org/wiki/xacro">
-  <xacro:include filename="$(find gp12_gazebo)/urdf/common_colors.xacro"/>
+  <xacro:include filename="$(find gp12_simulation)/urdf/common_colors.xacro"/>
   <xacro:macro name="material_yaskawa_blue">
     <material name="">

File: src/gp12_simulation/urdf/gp12.xacro (robot description, xacro)
@@ -1,12 +1,5 @@
 <?xml version="1.0" ?>
 <robot name="motoman_gp12" xmlns:xacro="http://ros.org/wiki/xacro">
-    <xacro:include filename="$(find gp12_gazebo)/urdf/gp12_macro.xacro" />
+    <xacro:include filename="$(find gp12_simulation)/urdf/gp12_macro.xacro" />
     <xacro:motoman_gp12 prefix=""/>
-    <gazebo>
-      <plugin name="gazebo_ros2_control" filename="libgazebo_ros2_control.so">
-        <robotNamespace>/</robotNamespace>
-        <verbose>true</verbose>
-        <parameters>$(find gp12_gazebo)/config/gp12_controllers.yaml</parameters>
-      </plugin>
-    </gazebo>
 </robot>

File: src/gp12_simulation/urdf/gp12_macro.xacro (robot description, xacro)
@@ -2,5 +2,5 @@
 <robot xmlns:xacro="http://ros.org/wiki/xacro">
 <xacro:macro name="motoman_gp12" params="prefix">
-    <xacro:include filename="$(find gp12_gazebo)/urdf/common_materials.xacro"/>
+    <xacro:include filename="$(find gp12_simulation)/urdf/common_materials.xacro"/>
     <!-- link list -->
     <link name="${prefix}base_link">
@@ -12,5 +12,5 @@
         <visual>
             <geometry>
-                <mesh filename="package://gp12_gazebo/meshes/visual/gp12_base_link.stl"/>
+                <mesh filename="package://gp12_simulation/meshes/visual/gp12_base_link.stl"/>
             </geometry>
             <xacro:material_yaskawa_blue/>
@@ -18,5 +18,5 @@
         <collision>
             <geometry>
-                <mesh filename="package://gp12_gazebo/meshes/collision/gp12_base_link.stl"/>
+                <mesh filename="package://gp12_simulation/meshes/collision/gp12_base_link.stl"/>
             </geometry>
         </collision>
@@ -30,5 +30,5 @@
         <visual>
             <geometry>
-                <mesh filename="package://gp12_gazebo/meshes/visual/gp12_link_1_s.stl"/>
+                <mesh filename="package://gp12_simulation/meshes/visual/gp12_link_1_s.stl"/>
             </geometry>
             <xacro:material_yaskawa_blue/>
@@ -36,5 +36,5 @@
         <collision>
             <geometry>
-                <mesh filename="package://gp12_gazebo/meshes/collision/gp12_link_1_s.stl"/>
+                <mesh filename="package://gp12_simulation/meshes/collision/gp12_link_1_s.stl"/>
             </geometry>
         </collision>
@@ -48,5 +48,5 @@
         <visual>
             <geometry>
-                <mesh filename="package://gp12_gazebo/meshes/visual/gp12_link_2_l.stl"/>
+                <mesh filename="package://gp12_simulation/meshes/visual/gp12_link_2_l.stl"/>
             </geometry>
             <xacro:material_yaskawa_blue/>
@@ -54,5 +54,5 @@
         <collision>
             <geometry>
-                <mesh filename="package://gp12_gazebo/meshes/collision/gp12_link_2_l.stl"/>
+                <mesh filename="package://gp12_simulation/meshes/collision/gp12_link_2_l.stl"/>
             </geometry>
         </collision>
@@ -66,5 +66,5 @@
         <visual>
             <geometry>
-                <mesh filename="package://gp12_gazebo/meshes/visual/gp12_link_3_u.stl"/>
+                <mesh filename="package://gp12_simulation/meshes/visual/gp12_link_3_u.stl"/>
             </geometry>
             <xacro:material_yaskawa_blue/>
@@ -72,5 +72,5 @@
         <collision>
             <geometry>
-                <mesh filename="package://gp12_gazebo/meshes/collision/gp12_link_3_u.stl"/>
+                <mesh filename="package://gp12_simulation/meshes/collision/gp12_link_3_u.stl"/>
             </geometry>
         </collision>
@@ -84,5 +84,5 @@
         <visual>
             <geometry>
-                <mesh filename="package://gp12_gazebo/meshes/visual/gp12_link_4_r.stl"/>
+                <mesh filename="package://gp12_simulation/meshes/visual/gp12_link_4_r.stl"/>
             </geometry>
             <xacro:material_yaskawa_blue/>
@@ -90,5 +90,5 @@
         <collision>
             <geometry>
-                <mesh filename="package://gp12_gazebo/meshes/collision/gp12_link_4_r.stl"/>
+                <mesh filename="package://gp12_simulation/meshes/collision/gp12_link_4_r.stl"/>
             </geometry>
         </collision>
@@ -102,5 +102,5 @@
         <visual>
             <geometry>
-                <mesh filename="package://gp12_gazebo/meshes/visual/gp12_link_5_b.stl"/>
+                <mesh filename="package://gp12_simulation/meshes/visual/gp12_link_5_b.stl"/>
             </geometry>
             <xacro:material_yaskawa_blue/>
@@ -108,5 +108,5 @@
         <collision>
             <geometry>
-                <mesh filename="package://gp12_gazebo/meshes/collision/gp12_link_5_b.stl"/>
+                <mesh filename="package://gp12_simulation/meshes/collision/gp12_link_5_b.stl"/>
             </geometry>
         </collision>
@@ -120,5 +120,5 @@
         <visual>
             <geometry>
-                <mesh filename="package://gp12_gazebo/meshes/visual/gp12_link_6_t.stl"/>
+                <mesh filename="package://gp12_simulation/meshes/visual/gp12_link_6_t.stl"/>
             </geometry>
             <xacro:material_yaskawa_blue/>
@@ -126,5 +126,5 @@
         <collision>
             <geometry>
-                <mesh filename="package://gp12_gazebo/meshes/collision/gp12_link_6_t.stl"/>
+                <mesh filename="package://gp12_simulation/meshes/collision/gp12_link_6_t.stl"/>
             </geometry>
         </collision>
@@ -174,46 +174,4 @@
         <limit lower="-7.9412" upper="7.9412" effort="33.30" velocity="12.2143"/>
     </joint>
-     <ros2_control name="GP12System" type="system">
-      <hardware>
-        <plugin>gazebo_ros2_control/GazeboSystem</plugin>
-      </hardware>
-        <joint name="${prefix}joint_1_s">
-            <command_interface name="position"/>
-            <state_interface name="position"/>
-            <state_interface name="velocity"/>
-            <state_interface name="effort"/>
-        </joint>
-        <joint name="${prefix}joint_2_l">
-            <command_interface name="position"/>
-            <state_interface name="position"/>
-            <state_interface name="velocity"/>
-            <state_interface name="effort"/>
-        </joint>
-        <joint name="${prefix}joint_3_u">
-            <command_interface name="position"/>
-            <state_interface name="position"/>
-            <state_interface name="velocity"/>
-            <state_interface name="effort"/>
-        </joint>
-        <joint name="${prefix}joint_4_r">
-            <command_interface name="position"/>
-            <state_interface name="position"/>
-            <state_interface name="velocity"/>
-            <state_interface name="effort"/>
-        </joint>
-        <joint name="${prefix}joint_5_b">
-            <command_interface name="position"/>
-            <state_interface name="position"/>
-            <state_interface name="velocity"/>
-            <state_interface name="effort"/>
-        </joint>
-        <joint name="${prefix}joint_6_t">
-            <command_interface name="position"/>
-            <state_interface name="position"/>
-            <state_interface name="velocity"/>
-            <state_interface name="effort"/>
-        </joint>
-    </ros2_control>
-    <!-- end of joint list -->
     <!-- ROS base_link to Robot Manufacturer World Coordinates transform -->
     <link name="${prefix}base" />
