Commit message: moveIt Issue solved

File: src/gp12_simulation/urdf/gp12.urdf (robot description, URDF)
Before this commit: robot motoman_gp12, 21 links, 20 joints
Links:
- link base: geometry visual box size=0.01 0.01 0.01
- link flange: geometry visual box size=0.01 0.01 0.01
- link tool0: geometry visual box size=0.01 0.01 0.01

File: src/gp12_simulation/urdf/gp12.xacro (robot description, xacro)
@@ -4,7 +4,7 @@
     <xacro:include filename="$(find gp12_simulation)/urdf/robotiq_2f_140.xacro" />
     <xacro:motoman_gp12 prefix=""/>
-    <!-- Attach Robotiq 2F-140 gripper to the robot tool0 frame -->
+    <!-- attach gripper -->
     <xacro:robotiq_2f_140 parent="tool0" tf_prefix="">
-      <origin xyz="0 0 0" rpy="0 0 0"/>
+        <origin xyz="0 0 0" rpy="0 0 0"/>
     </xacro:robotiq_2f_140>
 </robot>

File: src/gp12_simulation/urdf/gp12_macro.xacro (robot description, xacro)
@@ -175,5 +175,10 @@
     </joint>
     <!-- ROS base_link to Robot Manufacturer World Coordinates transform -->
-    <link name="${prefix}base" />
+    <link name="${prefix}base">
+        <visual>
+            <geometry><box size="0.01 0.01 0.01"/></geometry>
+            <xacro:material_yaskawa_blue/>
+        </visual>
+    </link>
     <joint name="${prefix}base_link-base" type="fixed">
         <origin xyz="0 0 0.450" rpy="0 0 0"/>
@@ -182,5 +187,10 @@
     </joint>
     <!-- ROS-Industrial 'flange' frame: attachment point for EEF models -->
-    <link name="${prefix}flange"/>
+    <link name="${prefix}flange">
+        <visual>
+            <geometry><box size="0.01 0.01 0.01"/></geometry>
+            <xacro:material_yaskawa_blue/>
+        </visual>
+    </link>
     <joint name="${prefix}joint_6_t-flange" type="fixed">
       <origin xyz="0.100 0 0" rpy="0 0 0"/>
@@ -189,5 +199,10 @@
     </joint>
     <!-- ROS-Industrial 'tool0' frame: all-zeros tool frame -->
-    <link name="${prefix}tool0"/>
+    <link name="${prefix}tool0">
+        <visual>
+            <geometry><box size="0.01 0.01 0.01"/></geometry>
+            <xacro:material_yaskawa_blue/>
+        </visual>
+    </link>
     <joint name="${prefix}flange-tool0" type="fixed">
       <origin xyz="0 0 0" rpy="3.1415926 -1.570796 0"/>
