Commit message: given actual meshes to package

File: ROS_packages/src/gp_12_trail/urdf/common_materials.xacro (robot description, xacro)
@@ -1,5 +1,5 @@
 <?xml version="1.0" ?>
 <robot xmlns:xacro="http://ros.org/wiki/xacro">
-  <xacro:include filename="$(find gp12_simulation)/urdf/common_colors.xacro"/>
+  <xacro:include filename="$(find gp_12_trail)/urdf/common_colors.xacro"/>
   <xacro:macro name="material_yaskawa_blue">
     <material name="">

File: ROS_packages/src/gp_12_trail/urdf/gp12.xacro (robot description, xacro)
@@ -1,6 +1,6 @@
 <?xml version="1.0" ?>
 <robot name="motoman_gp12" xmlns:xacro="http://ros.org/wiki/xacro">
-    <xacro:include filename="$(find gp12_simulation)/urdf/gp12_macro.xacro" />
-    <xacro:include filename="$(find gp12_simulation)/urdf/robotiq_2f_140.xacro" />
+    <xacro:include filename="$(find gp_12_trail)/urdf/gp12_macro.xacro" />
+    <xacro:include filename="$(find gp_12_trail)/urdf/robotiq_2f_140.xacro" />
     <xacro:motoman_gp12 prefix=""/>
     <!-- attach gripper -->

File: ROS_packages/src/gp_12_trail/urdf/gp12_gripper.xacro (robot description, xacro)
@@ -2,5 +2,5 @@
 <robot name="robotiq_test" xmlns:xacro="http://ros.org/wiki/xacro">
   <!-- include gripper -->
-  <xacro:include filename="$(find gp12_simulation)/urdf/robotiq_2f_140.xacro"/>
+  <xacro:include filename="$(find gp_12_trail)/urdf/robotiq_2f_140.xacro"/>
   <!-- world -->
   <link name="world"/>

File: ROS_packages/src/gp_12_trail/urdf/gp12_macro.xacro (robot description, xacro)
@@ -2,5 +2,5 @@
 <robot xmlns:xacro="http://ros.org/wiki/xacro">
 <xacro:macro name="motoman_gp12" params="prefix">
-    <xacro:include filename="$(find gp12_simulation)/urdf/common_materials.xacro"/>
+    <xacro:include filename="$(find gp_12_trail)/urdf/common_materials.xacro"/>
     <!-- link list -->
     <link name="${prefix}base_link">
@@ -12,11 +12,11 @@
         <visual>
             <geometry>
-                <mesh filename="package://gp12_simulation/meshes/visual/gp12_base_link.stl"/>
-            </geometry>
-            <xacro:material_yaskawa_blue/>
-        </visual>
-        <collision>
-            <geometry>
-                <mesh filename="package://gp12_simulation/meshes/collision/gp12_base_link.stl"/>
+                <mesh filename="package://gp_12_trail/meshes/visual/gp12_base_link.stl"/>
+            </geometry>
+            <xacro:material_yaskawa_blue/>
+        </visual>
+        <collision>
+            <geometry>
+                <mesh filename="package://gp_12_trail/meshes/collision/gp12_base_link.stl"/>
             </geometry>
         </collision>
@@ -30,11 +30,11 @@
         <visual>
             <geometry>
-                <mesh filename="package://gp12_simulation/meshes/visual/gp12_link_1_s.stl"/>
-            </geometry>
-            <xacro:material_yaskawa_blue/>
-        </visual>
-        <collision>
-            <geometry>
-                <mesh filename="package://gp12_simulation/meshes/collision/gp12_link_1_s.stl"/>
+                <mesh filename="package://gp_12_trail/meshes/visual/gp12_link_1_s.stl"/>
+            </geometry>
+            <xacro:material_yaskawa_blue/>
+        </visual>
+        <collision>
+            <geometry>
+                <mesh filename="package://gp_12_trail/meshes/collision/gp12_link_1_s.stl"/>
             </geometry>
         </collision>
@@ -48,11 +48,11 @@
         <visual>
             <geometry>
-                <mesh filename="package://gp12_simulation/meshes/visual/gp12_link_2_l.stl"/>
-            </geometry>
-            <xacro:material_yaskawa_blue/>
-        </visual>
-        <collision>
-            <geometry>
-                <mesh filename="package://gp12_simulation/meshes/collision/gp12_link_2_l.stl"/>
+                <mesh filename="package://gp_12_trail/meshes/visual/gp12_link_2_l.stl"/>
+            </geometry>
+            <xacro:material_yaskawa_blue/>
+        </visual>
+        <collision>
+            <geometry>
+                <mesh filename="package://gp_12_trail/meshes/collision/gp12_link_2_l.stl"/>
             </geometry>
         </collision>
@@ -66,11 +66,11 @@
         <visual>
             <geometry>
-                <mesh filename="package://gp12_simulation/meshes/visual/gp12_link_3_u.stl"/>
-            </geometry>
-            <xacro:material_yaskawa_blue/>
-        </visual>
-        <collision>
-            <geometry>
-                <mesh filename="package://gp12_simulation/meshes/collision/gp12_link_3_u.stl"/>
+                <mesh filename="package://gp_12_trail/meshes/visual/gp12_link_3_u.stl"/>
+            </geometry>
+            <xacro:material_yaskawa_blue/>
+        </visual>
+        <collision>
+            <geometry>
+                <mesh filename="package://gp_12_trail/meshes/collision/gp12_link_3_u.stl"/>
             </geometry>
         </collision>
@@ -84,11 +84,11 @@
         <visual>
             <geometry>
-                <mesh filename="package://gp12_simulation/meshes/visual/gp12_link_4_r.stl"/>
-            </geometry>
-            <xacro:material_yaskawa_blue/>
-        </visual>
-        <collision>
-            <geometry>
-                <mesh filename="package://gp12_simulation/meshes/collision/gp12_link_4_r.stl"/>
+                <mesh filename="package://gp_12_trail/meshes/visual/gp12_link_4_r.stl"/>
+            </geometry>
+            <xacro:material_yaskawa_blue/>
+        </visual>
+        <collision>
+            <geometry>
+                <mesh filename="package://gp_12_trail/meshes/collision/gp12_link_4_r.stl"/>
             </geometry>
         </collision>
@@ -102,11 +102,11 @@
         <visual>
             <geometry>
-                <mesh filename="package://gp12_simulation/meshes/visual/gp12_link_5_b.stl"/>
-            </geometry>
-            <xacro:material_yaskawa_blue/>
-        </visual>
-        <collision>
-            <geometry>
-                <mesh filename="package://gp12_simulation/meshes/collision/gp12_link_5_b.stl"/>
+                <mesh filename="package://gp_12_trail/meshes/visual/gp12_link_5_b.stl"/>
+            </geometry>
+            <xacro:material_yaskawa_blue/>
+        </visual>
+        <collision>
+            <geometry>
+                <mesh filename="package://gp_12_trail/meshes/collision/gp12_link_5_b.stl"/>
             </geometry>
         </collision>
@@ -120,11 +120,11 @@
         <visual>
             <geometry>
-                <mesh filename="package://gp12_simulation/meshes/visual/gp12_link_6_t.stl"/>
-            </geometry>
-            <xacro:material_yaskawa_blue/>
-        </visual>
-        <collision>
-            <geometry>
-                <mesh filename="package://gp12_simulation/meshes/collision/gp12_link_6_t.stl"/>
+                <mesh filename="package://gp_12_trail/meshes/visual/gp12_link_6_t.stl"/>
+            </geometry>
+            <xacro:material_yaskawa_blue/>
+        </visual>
+        <collision>
+            <geometry>
+                <mesh filename="package://gp_12_trail/meshes/collision/gp12_link_6_t.stl"/>
             </geometry>
         </collision>

File: ROS_packages/src/gp_12_trail/urdf/robotiq_2f_140.xacro (robot description, xacro)
@@ -2,5 +2,5 @@
 <robot xmlns:xacro="http://ros.org/wiki/xacro">
   <!-- Include the gripper macro implementation -->
-  <xacro:include filename="$(find gp12_simulation)/urdf/robotiq_2f_140_macro.xacro"/>
+  <xacro:include filename="$(find gp_12_trail)/urdf/robotiq_2f_140_macro.xacro"/>
   <!-- Macro that attaches gripper to a parent link -->
   <xacro:macro name="robotiq_2f_140" params="parent tf_prefix *origin">

File: ROS_packages/src/gp_12_trail/urdf/robotiq_2f_140_macro.xacro (robot description, xacro)
@@ -1,5 +1,5 @@
 <?xml version="1.0"?>
 <robot xmlns:xacro="http://ros.org/wiki/xacro">
-  <xacro:include filename="$(find gp12_simulation)/urdf/robotiq_arg2f_transmission.xacro" />
+  <xacro:include filename="$(find gp_12_trail)/urdf/robotiq_arg2f_transmission.xacro" />
   <xacro:macro name="outer_knuckle" params="prefix fingerprefix stroke">
     <link name="${prefix}${fingerprefix}_outer_knuckle">
@@ -18,5 +18,5 @@
         <origin xyz="0 0 0" rpy="0 0 0" />
         <geometry>
-          <mesh filename="package://gp12_simulation/meshes/visual/robotiq_arg2f_${stroke}_outer_knuckle.stl" />
+          <mesh filename="package://gp_12_trail/meshes/visual/robotiq_arg2f_${stroke}_outer_knuckle.stl" />
         </geometry>
         <material name="">
@@ -27,5 +27,5 @@
         <origin xyz="0 0 0" rpy="0 0 0" />
         <geometry>
-          <mesh filename="package://gp12_simulation/meshes/collision/robotiq_arg2f_${stroke}_outer_knuckle.stl" />
+          <mesh filename="package://gp_12_trail/meshes/collision/robotiq_arg2f_${stroke}_outer_knuckle.stl" />
         </geometry>
       </collision>
@@ -48,5 +48,5 @@
         <origin xyz="0 0 0" rpy="0 0 0" />
         <geometry>
-          <mesh filename="package://gp12_simulation/meshes/visual/robotiq_arg2f_${stroke}_outer_finger.stl" />
+          <mesh filename="package://gp_12_trail/meshes/visual/robotiq_arg2f_${stroke}_outer_finger.stl" />
         </geometry>
         <material name="">
@@ -57,5 +57,5 @@
         <origin xyz="0 0 0" rpy="0 0 0" />
         <geometry>
-          <mesh filename="package://gp12_simulation/meshes/collision/robotiq_arg2f_${stroke}_outer_finger.stl" />
+          <mesh filename="package://gp_12_trail/meshes/collision/robotiq_arg2f_${stroke}_outer_finger.stl" />
         </geometry>
       </collision>
@@ -78,5 +78,5 @@
         <origin xyz="0 0 0" rpy="0 0 0" />
         <geometry>
-          <mesh filename="package://gp12_simulation/meshes/visual/robotiq_arg2f_${stroke}_inner_knuckle.stl" />
+          <mesh filename="package://gp_12_trail/meshes/visual/robotiq_arg2f_${stroke}_inner_knuckle.stl" />
         </geometry>
         <material name="">
@@ -87,5 +87,5 @@
         <origin xyz="0 0 0" rpy="0 0 0" />
         <geometry>
-          <mesh filename="package://gp12_simulation/meshes/collision/robotiq_arg2f_${stroke}_inner_knuckle.stl" />
+          <mesh filename="package://gp_12_trail/meshes/collision/robotiq_arg2f_${stroke}_inner_knuckle.stl" />
         </geometry>
       </collision>
@@ -108,5 +108,5 @@
         <origin xyz="0 0 0" rpy="0 0 0" />
         <geometry>
-          <mesh filename="package://gp12_simulation/meshes/visual/robotiq_arg2f_${stroke}_inner_finger.stl" />
+          <mesh filename="package://gp_12_trail/meshes/visual/robotiq_arg2f_${stroke}_inner_finger.stl" />
         </geometry>
         <material name="">
@@ -117,5 +117,5 @@
         <origin xyz="0 0 0" rpy="0 0 0" />
         <geometry>
-          <mesh filename="package://gp12_simulation/meshes/collision/robotiq_arg2f_${stroke}_inner_finger.stl" />
+          <mesh filename="package://gp_12_trail/meshes/collision/robotiq_arg2f_${stroke}_inner_finger.stl" />
         </geometry>
       </collision>
@@ -181,5 +181,5 @@
     </joint>
   </xacro:macro>
-  <xacro:include filename="$(find gp12_simulation)/urdf/robotiq_arg2f.xacro" />
+  <xacro:include filename="$(find gp_12_trail)/urdf/robotiq_arg2f.xacro" />
   <xacro:macro name="finger_joint" params="prefix">
     <joint name="${prefix}finger_joint" type="revolute">

File: ROS_packages/src/gp_12_trail/urdf/robotiq_arg2f.xacro (robot description, xacro)
@@ -11,5 +11,5 @@
         <origin xyz="0 0 0" rpy="0 0 0" />
         <geometry>
-          <mesh filename="package://gp12_simulation/meshes/visual/robotiq_arg2f_base_link.stl" />
+          <mesh filename="package://gp_12_trail/meshes/visual/robotiq_arg2f_base_link.stl" />
         </geometry>
         <material name="">
@@ -20,5 +20,5 @@
         <origin xyz="0 0 0" rpy="0 0 0" />
         <geometry>
-          <mesh filename="package://gp12_simulation/meshes/collision/robotiq_arg2f_base_link.stl" />
+          <mesh filename="package://gp_12_trail/meshes/collision/robotiq_arg2f_base_link.stl" />
         </geometry>
       </collision>
