Commit message: typo

File: ROS_packages/src/gp_12_trail/urdf/gp12.urdf (robot description, URDF)
Before this commit: robot motoman_gp12, 21 links, 20 joints
Links:
- link base_link: geometry collision mesh filename=package://gp_12_trail/meshes/collision/gp12_base_link.stl; visual mesh filename=package://gp_12_trail/meshes/visual/gp12_base_link.stl
- link left_inner_finger: geometry collision mesh filename=package://gp_12_trail/meshes/collision/robotiq_arg2f_140_in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; visual mesh filename=package://gp_12_trail/meshes/visual/robotiq_arg2f_140_inner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
- link left_inner_knuckle: geometry collision mesh filename=package://gp_12_trail/meshes/collision/robotiq_arg2f_140_in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; visual mesh filename=package://gp_12_trail/meshes/visual/robotiq_arg2f_140_inner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
- link left_outer_finger: geometry collision mesh filename=package://gp_12_trail/meshes/collision/robotiq_arg2f_140_ou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; visual mesh filename=package://gp_12_trail/meshes/visual/robotiq_arg2f_140_outer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
- link left_outer_knuckle: geometry collision mesh filename=package://gp_12_trail/meshes/collision/robotiq_arg2f_140_ou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; visual mesh filename=package://gp_12_trail/meshes/visual/robotiq_arg2f_140_outer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
- link link_1_s: geometry collision mesh filename=package://gp_12_trail/meshes/collision/gp12_link_1_s.stl; visual mesh filename=package://gp_12_trail/meshes/visual/gp12_link_1_s.stl
- link link_2_l: geometry collision mesh filename=package://gp_12_trail/meshes/collision/gp12_link_2_l.stl; visual mesh filename=package://gp_12_trail/meshes/visual/gp12_link_2_l.stl
- link link_3_u: geometry collision mesh filename=package://gp_12_trail/meshes/collision/gp12_link_3_u.stl; visual mesh filename=package://gp_12_trail/meshes/visual/gp12_link_3_u.stl
- link link_4_r: geometry collision mesh filename=package://gp_12_trail/meshes/collision/gp12_link_4_r.stl; visual mesh filename=package://gp_12_trail/meshes/visual/gp12_link_4_r.stl
- link link_5_b: geometry collision mesh filename=package://gp_12_trail/meshes/collision/gp12_link_5_b.stl; visual mesh filename=package://gp_12_trail/meshes/visual/gp12_link_5_b.stl
- link link_6_t: geometry collision mesh filename=package://gp_12_trail/meshes/collision/gp12_link_6_t.stl; visual mesh filename=package://gp_12_trail/meshes/visual/gp12_link_6_t.stl
- link right_inner_finger: geometry collision mesh filename=package://gp_12_trail/meshes/collision/robotiq_arg2f_140_in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; visual mesh filename=package://gp_12_trail/meshes/visual/robotiq_arg2f_140_inner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
- link right_inner_knuckle: geometry collision mesh filename=package://gp_12_trail/meshes/collision/robotiq_arg2f_140_in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; visual mesh filename=package://gp_12_trail/meshes/visual/robotiq_arg2f_140_inner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
- link right_outer_finger: geometry collision mesh filename=package://gp_12_trail/meshes/collision/robotiq_arg2f_140_ou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; visual mesh filename=package://gp_12_trail/meshes/visual/robotiq_arg2f_140_outer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
- link right_outer_knuckle: geometry collision mesh filename=package://gp_12_trail/meshes/collision/robotiq_arg2f_140_ou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; visual mesh filename=package://gp_12_trail/meshes/visual/robotiq_arg2f_140_outer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
- link robotiq_arg2f_base_link: geometry collision mesh filename=package://gp_12_trail/meshes/collision/robotiq_arg2f_base_l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; visual mesh filename=package://gp_12_trail/meshes/visual/robotiq_arg2f_base_link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
